File: zynthian_allinone/zynthian_allinone.sch (KiCad schematic (older format))
At the start: 31 parts

Commit message: Random playing
Parts:
- removed C1, C2, C3: 100n, Capacitors_ThroughHole:C_Disc_D3.0mm_W1.6mm_P2.50mm, symbol C
- removed D1, D3, D4: 1N4148, Discret:D3, symbol D
- removed D2: 1N5819, Discret:D4, symbol D
- removed MIDI-1: MIDI-IN, Connectors_JST:JST_XH_B04B-XH-A_04x2.50mm_Straight, symbol CONN_01X04_MALE
- removed MIDI-2: MIDI-THRU, Connectors_JST:JST_XH_B04B-XH-A_04x2.50mm_Straight, symbol CONN_01X04_MALE
- removed MIDI-3: MIDI-OUT, Connectors_JST:JST_XH_B04B-XH-A_04x2.50mm_Straight, symbol CONN_01X04_MALE
- removed OC1, OC2, OC3: H11L1, Housings_DIP:DIP-6_W7.62mm, symbol H11L1
- removed R1: 100, Discret:R4, symbol R
- removed R10: 10K, Discret:R4, symbol R
- removed R2, R6, R8: 470, Discret:R4, symbol R
- removed R3, R4, R9: 1K, Discret:R4, symbol R
- removed R5, R7: 4K7, Discret:R4, symbol R
- removed SW-1: SW1, Connectors_JST:JST_XH_B05B-XH-A_05x2.50mm_Straight, symbol CONN_01X05
- C4: symbol C -> zynthian_allinone-rescue:C
- CTRL-1, CTRL-2, CTRL-3, CTRL-4: symbol CONN_01X04_MALE -> zynthian_allinone-rescue:CONN_01X04_MALE
- MCP23017: symbol MCP23017 -> zynthian_allinone-rescue:MCP23017
- RBPi-1: symbol CONN_02X20 -> zynthian_allinone-rescue:CONN_02X20
Connections:
- net MIDI-IN: no longer names the net of RBPi-1.10 (P10)
- net MIDI-OUT: no longer names the net of RBPi-1.8 (P8)
